File: final_kicad/final_kicad.kicad_sch (KiCad schematic)
At the start: 72 parts, among them J3 Reflectance Sensor Array, M1 Motor, M3 Servo for Side Indicator, M4 Servo for Joint 1, M5 Motor_Step_4Wire, M6 Motor for Linear Actuator, M7 Servo for Joint 2, Q1 Photo_NPN, Q2 MOSFET-N, SW1 Reset, SW2 Reset, U1 SN754410, U2 MCP6294, U2 PIC32MX170F256B, U4 Comparator, U5 L293NE, U6 L293NE

Commit message: final KiCAD update
Parts:
- removed D19, D20, D21, D22: Bi-color LED, symbol ME218_BaseLib:LED
- removed D27: LED, symbol ME218_BaseLib:LED
- removed R11, R12: 200 Ohm, symbol ME218_BaseLib:Res1
- added C11: 0.1uF, symbol ME218_BaseLib:Cap
- added R_pull1, R_pull10, R_pull2, R_pull3, R_pull4, R_pull5, R_pull6, R_pull7, R_pull8, R_pull9: 10k, symbol ME218_BaseLib:Res1
- U2: value MCP6294 -> MCP6294 Op-Amp
Connections:
- net left_IR is gone; now on net DO: U2.10 (RA3)
- net right_IR is gone; now on net DO: U2.25 (RB14)
- net +3.3V: now also J3.8 (Pin_8); no longer M4.2 (+), M7.2 (+)
- net +5V: now also M4.2 (+), M7.2 (+), C11.2
- net +6V: no longer D15.2 (A), D16.1 (K), M5.2 (-), U5.6 (2Y)
- net BEACON_SENSOR: no longer R8.2, U4.1
- net DO: now also PIC0.7 (RB3); no longer U2.22 (RB11)
- net Earth: now also J3.7 (Pin_7), U4.11 (V-), C11.1
- net GND: now also R_pull1.2, R_pull10.2, R_pull2.2, R_pull3.2, R_pull4.2, R_pull5.2, R_pull6.2, R_pull7.2, R_pull8.2, R_pull9.2
- net OC3: now also R_pull7.1
- net at PIC0.22 (RB11), U5.10 (3A): now also R_pull4.1
- net at PIC0.23 (RB12), U5.15 (4A): now also R_pull1.1
- net at PIC0.18 (PGED2/5VT/RB9), U5.2 (1A): now also R_pull3.1
- net at PIC0.21 (PGEC2/5VT/RB10), U5.7 (2A): now also R_pull2.1
- net at D24.2 (A), D26.1 (K), M6.1 (+)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: now also R_pull9.1
- net at D23.2 (A), D25.1 (K), M6.2 (-)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: now also R_pull10.1
- net at U1.10 (3A), U2.18 (PGED2/5VT/RB9): now also R_pull8.1
- net at U1.2 (1A), U2.14 (PGED3/5VT/RB5): now also R_pull6.1
- net OC1 renamed OC4
- net OC4: now also R_pull5.1
- net button: no longer names the net of PIC0.6 (RB2)
- new net: D15.2 (A), D16.1 (K), M5.2 (-), U5.6 (2Y)
- new net BEACON_SENSOR_OUTPUT: R8.2, U4.1
Other:
- note added: "(Left of Cart)"
- note added: "(Right of Cart)"
- note added: "IR Sensor Module"
- note added: "Linear Stage"
- note removed: "For Linear Stage"
- moved on the sheet: C5, C6, C7, C8, C9, M1, M3, M4, M5, M6, M7, PIC0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

Commit message: up
Parts:
- removed J3: Reflectance Sensor Array, symbol ME218_BaseLib:Molex8
Connections:
- net GND: no longer C1.2, C10.1, C2.2, C3.1, C4.2, C5.2, C6.2, C7.1, C8.2, C9.1, D10.1 (K), D12.2 (A), D14.2 (A), D16.2 (A), D18.2 (A), D9.1 (K), M3.3 (-), M4.3 (-), M7.3 (-), PIC0.19 (Vss), PIC0.27 (AVss), PIC0.8 (Vss), R_pull.2, R_pull1.2, R_pull10.2, R_pull2.2, R_pull3.2, R_pull4.2, R_pull5.2, R_pull6.2, R_pull7.2, R_pull8.2, R_pull9.2, SW1.2, SW2.2, U2.19 (Vss), U2.27 (AVss), U2.8 (Vss), U5.12 (GND), U5.13 (GND), U5.4 (GND), U5.5 (GND), U6.12 (GND), U6.13 (GND), U6.4 (GND), U6.5 (GND), U6.9 (EN3,4)
- removed net DO: PIC0.7 (RB3), U2.10 (RA3), U2.25 (RB14)
- new net GNDREF: C1.2, C10.1, C2.2, C3.1, C4.2, C5.2, C6.2, C7.1, C8.2, C9.1, D10.1 (K), D12.2 (A), D14.2 (A), D16.2 (A), D18.2 (A), D9.1 (K), M3.3 (-), M4.3 (-), M7.3 (-), PIC0.19 (Vss), PIC0.27 (AVss), PIC0.8 (Vss), R_pull.2, R_pull1.2, R_pull10.2, R_pull2.2, R_pull3.2, R_pull4.2, R_pull5.2, R_pull6.2, R_pull7.2, R_pull8.2, R_pull9.2, SW1.2, SW2.2, U2.19 (Vss), U2.27 (AVss), U2.8 (Vss), U5.12 (GND), U5.13 (GND), U5.4 (GND), U5.5 (GND), U6.12 (GND), U6.13 (GND), U6.4 (GND), U6.5 (GND), U6.9 (EN3,4)
Other:
- note added: "(placed on leftside)"
- note added: "(placed on rightside)"
- note added: "A0"
- note added: "A1"
- note added: "A2"
- note added: "A3"
- note added: "A4"
- note added: "A5"
- note added: "A6"
- note added: "A7"
- note added: "A8"
- note added: "D0"
- note added: "GND"
- note added: "Reflectance Sensor Array"
- note added: "Vcc"
- note removed: "(Left of Cart)"
- note removed: "(Right of Cart)"
- note removed: "Analog Readings"
- moved on the sheet: M7

Commit message: replace lab8 H-bridge with project H-bridge
Parts:
- removed C10, C9: 0.1uF, symbol ME218_BaseLib:Cap
- removed D1 (x3), D11, D12, D13, D14, D15, D16, D17, D18, D2 (x3), D23, D24, D25, D26, D5, D6: Diode, symbol ME218_BaseLib:Diode
- removed R_pull10, R_pull9: 10k, symbol ME218_BaseLib:Res1
- removed U1: SN754410, Package_DIP:DIP-16_W7.62mm, symbol ME218_BaseLib:L293NE
- removed U5, U6: L293NE, Package_DIP:DIP-16_W7.62mm, symbol ME218_BaseLib:L293NE
- added R11: 1k, symbol ME218_BaseLib:Res1
- added R12: 10k, symbol ME218_BaseLib:Res1
- added SW3: Game Start Button, symbol ME218_BaseLib:SW_Push
- M6: value Motor for Linear Actuator -> Motor
Connections:
- net GND is gone; now on net GNDREF: PRG1.3 (Vss), PRG2.3 (Vss)
- net +3.3V: now also R12.2
- net +5V: no longer C11.2
- net Earth: no longer C11.1
- net GNDREF: now also C11.2, SW3.2
- net at M1.1 (+): now also M1.2 (-)
- net at PIC0.6 (RB2): now also R11.1
- new net: C11.1, R11.2, R12.1, SW3.1
- no-connect marks 0 -> 7
Other:
- note added: "+14.4V"
- note added: "EF"
- note added: "In1"
- note added: "In2"
- note added: "Left Wheel"
- note added: "Linear Actuator"
- note added: "OC1"
- note added: "OC2"
- note added: "OC3"
- note added: "OC4"
- note added: "Out1"
- note added: "Out2"
- note added: "Right Wheel"
- note added: "TLE 5206 H-bridge"
- note added: "Vs"
- note removed: "+5V from big power supply"
- note removed: "Channel 1"
- note removed: "Channel 2"
- note removed: "Channel 3"
- note removed: "Channel 4"
- note removed: "LEFT Motor"
- note removed: "RIGHT Motor"
- moved on the sheet: M1, Q2, R_limit, R_pull7, R_pull8

Commit message: final KiCAD
Parts:
- added R_pull10, R_pull9: 10k, symbol ME218_BaseLib:Res1
Connections:
- net GNDREF: now also R_pull10.2, R_pull9.2
- net at PIC0.2 (RA0): now also R_pull10.1
- net at PIC0.3 (RA1): now also R_pull9.1
- net at M1.1 (+): no longer M1.2 (-)
- no-connect marks 7 -> 11
